Commit message: use the name in the materials so multiple cameras can be on same tf tree

File: zed_wrapper/urdf/include/materials.urdf.xacro (robot description, xacro)
@@ -15,16 +15,20 @@
 OF THIS SOFTWARE, EVEN IF ADVISED OF THE POSSIBILITY OF SUCH DAMAGE.
 -->
-<robot>
-    <material name="zed_mat">
+<robot xmlns:xacro="http://ros.org/wiki/xacro">
+  <xacro:macro name="zed_mat" params="name">
+    <material name="${name}_zed_mat">
         <color rgba="0.8 0.8 0.8 0.8"/>
     </material>
-    <material name="zedm_mat">
+    <material name="${name}_zedm_mat">
         <color rgba="0 0 0 0.9"/>
     </material>
-    <material name="zed2_mat">
+    <material name="${name}_zed2_mat">
         <color rgba="0.25 0.25 0.25 0.99"/>
     </material>
-    <material name="zed2i_mat">
+    <material name="${name}_zed2i_mat">
         <color rgba="0.25 0.25 0.25 0.99"/>
     </material>
+    <!--
+    -->
+  </xacro:macro>
 </robot>

File: zed_wrapper/urdf/zed_macro.urdf.xacro (robot description, xacro)
@@ -26,4 +26,5 @@
   -->
   <xacro:macro name="zed_camera" params="name=zed model=zed parent *origin">
+    <xacro:zed_mat name="${name}" />
     <xacro:if value="${model == 'zed'}">
       <xacro:property name="baseline" value="0.12" />
@@ -68,5 +69,5 @@
           <mesh filename="package://zed_interfaces/meshes/${model}.stl" />
         </geometry>
-        <material name="${model}_mat" />
+        <material name="${name}_${model}_mat" />
       </visual>
       <collision>
